File: CosmosRpiDevBoard.kicad_pcb (KiCad board)
At the start: 4 copper layers, 85 x 56 mm, 151 parts, among them J1 RPi Connector, J2 ARJM11D7-009-AB-EW2, J3 UJ20-C-H-G-SMT-5-P16-TR, J4 MSD-4-A, J5 5V Fan, J6 3.3V Fan, J7 Ext Pins, J8 SW Debug, SW1 DS04-254-1L-03BK, SW2 TS02-66-43-BK-160-LCR-D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

Commit message: Update
Parts:
- moved C17 156.3 mm to (205.1, 68.2), turned to 180 degrees
- moved R4 153.5 mm to (200.0, 69.2), turned to 180 degrees
- moved C18 152.9 mm to (201.6, 71.2), turned to 90 degrees
- moved Y1 152.5 mm to (204.5, 71.1)
- moved C11 1.70 mm to (204.4, 82.6)
- moved C10 1.70 mm to (204.4, 80.2)
- moved C8 1.70 mm to (204.4, 79.0)
- moved C9 1.70 mm to (204.4, 81.4)
- moved R37 0.40 mm to (199.9, 72.9)
- moved R38 0.40 mm to (198.7, 72.9)
- moved C59 0.10 mm to (178.9, 88.3)
Routing:
- net ETH_RD+: track 17.5 -> 7.88 mm
- net /ETH_XO: track 0.00 -> 7.91 mm
- net /ETH_BIAS: track 0.00 -> 6.81 mm
- net ETH_RD-: track 18.0 -> 11.5 mm
- net ETH_RXD_0: track 25.9 -> 19.6 mm
- net ETH_TXD_0: track 13.3 -> 7.34 mm
- net /ETH_XI: track 0.00 -> 5.11 mm
- net +5V_RPi: track 0.00 -> 2.54 mm
- net ETH_TD+: track 11.6 -> 9.33 mm
- net /ETH_RX_ER: track 6.31 -> 5.03 mm
- net GND_CHS: vias 0 -> 20
- net GND: vias 23 -> 32
- added copper zone on F.Cu, net +3.3V
- added copper zone on F.Cu, net GND
- removed copper zone on B.Cu, net GND_CHS
Other:
- rule pad_to_mask_clearance: 0.1 -> 0.025

Commit message: Update
Parts:
- removed C16: 100n, Capacitor_SMD:C_1206_3216Metric
- removed R42, R43, R44, R45, R51: 33, Resistor_SMD:R_0402_1005Metric
- removed R5: 1M, Resistor_SMD:R_1206_3216Metric
- added C65: 6p, Capacitor_SMD:C_0402_1005Metric, F.Cu at (211.2, 87.6)
- added C66: 6p, Capacitor_SMD:C_0402_1005Metric, F.Cu at (217.1, 89.4)
- added G***: LOGO, LOGO, F.Cu at (216.6, 63.7)
- added Y6: 24MHz, Crystal:Crystal_SMD_3225-4Pin_3.2x2.5mm, F.Cu at (214.1, 89.5)
- U2: footprint PCB:PCB_Antenna -> RF_Antenna:Texas_SWRA117D_2.4GHz_Right
- moved R12 176.2 mm to (225.7, 65.2), turned to 90 degrees
- moved U9 173.8 mm to (211.0, 105.0)
- moved L1 173.6 mm to (215.0, 105.0), turned to 90 degrees
- moved C32 172.4 mm to (218.2, 104.4), turned to -90 degrees
- moved R20 170.7 mm to (220.0, 96.3), turned to 90 degrees
- moved R46 170.7 mm to (224.0, 113.0), turned to -90 degrees
- moved R13 170.4 mm to (218.8, 86.9), turned to 180 degrees
- moved C34 170.1 mm to (217.0, 104.4), turned to -90 degrees
- moved R21 169.5 mm to (220.0, 91.1), turned to -90 degrees
- moved D1 168.5 mm to (224.0, 110.0), turned to 90 degrees
- moved R49 166.1 mm to (221.0, 113.0), turned to -90 degrees
- moved U8 165.7 mm to (217.0, 93.6)
- moved C23 164.8 mm to (209.6, 97.2)
- moved D2 164.6 mm to (221.0, 110.0), turned to 90 degrees
- moved C24 164.5 mm to (209.6, 98.4)
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Connections:
- J2 pad SH1: GND_CHS -> GND
- J2 pad SH2: GND_CHS -> GND
- J3 pad S1: GND_CHS -> GND
- J4 pad 6: unconnected-(J4-VSS-Pad6) -> GND
- R1 pad 2: +5V -> +3.3V
- U2 pad 1: GND -> /ESP32_ANT_IN
- U2 pad 2: /ESP32_ANT_IN -> GND
- U3 pad 10: /STM32_SPI2_MISO -> SPI2_MISO
- U3 pad 22: /STM32_SPI1_MISO -> SPI1_MISO
- U3 pad 35: unconnected-(U3-PB14-Pad35) -> RPi_FAULT
- U3 pad 41: /STM32_USB_CLK -> RPi_CTRL
- U3 pad 58: unconnected-(U3-PB6-Pad58) -> STM32_LED
- U5 pad 12: /ESP32_SPI2_MOSI -> SPI2_MOSI
- U5 pad 16: /ESP32_SPI1_MOSI -> SPI1_MOSI
- U7 pad 21: unconnected-(U7-XTALOUT-Pad21) -> USB_CLK_OUT
- U7 pad 22: USB_CLK -> USB_CLK_IN
- U9 pad 3: unconnected-(U9-VIN-Pad3) -> +5V
Routing:
- net +3.3V: track 0.00 -> 412.7 mm, vias 8 -> 34
- net +5V: track 0.00 -> 184.4 mm, vias 0 -> 8
- net +5V_RPi: track 2.54 -> 135.2 mm, vias 0 -> 2
- net RPi_CTRL: track 0.00 -> 97.9 mm, vias 0 -> 6
- net RST_N: track 0.00 -> 96.8 mm, vias 0 -> 4
- net ESP32_D-: track 0.00 -> 80.0 mm, vias 0 -> 2
- net STM32_WKUP: track 0.00 -> 78.8 mm, vias 0 -> 2
- net ESP32_D+: track 0.00 -> 77.9 mm, vias 0 -> 2
- net ESP32_LED: track 0.00 -> 64.4 mm, vias 0 -> 2
- net STM32_BOOT: track 0.00 -> 59.3 mm, vias 0 -> 2
- net SD_DAT2: track 0.00 -> 59.3 mm, vias 0 -> 2
- net SD_DAT3: track 0.00 -> 55.2 mm, vias 0 -> 2
- net RPi_FAULT: track 0.00 -> 52.6 mm, vias 0 -> 2
- net STM32_LED: track 0.00 -> 51.6 mm, vias 0 -> 2
- net SPI2_CLK: track 0.00 -> 50.7 mm, vias 0 -> 2
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- added copper zone on F.Cu, net +5V
- added copper zone on F.Cu, net +5V_RPi
- added copper zone on B.Cu, net GND
- added copper zone on In2.Cu, net GND
- removed copper zone on In2.Cu, net +3.3V
- removed copper zone on In1.Cu, net GND_CHS
- removed copper zone on In2.Cu, net GND_CHS
Other:
- board size 85 x 56 mm -> 90.4 x 56 mm
- board text added: "+"
- board text added: "-"
- board text added: "PWM"
