File: CosmosRpiDevBoard.kicad_sch (KiCad schematic)
At the start: 12 parts, among them J1 RPi Connector, SW1 DS04-254-1L-01BK, U1 AP22814AW5, U2 TC7WB66CFK, U3 TC7WB66CFK, U4 TC7WB66CFK, U5 TC7WB66CFK

Commit message: Update
Parts:
- removed U2, U3, U4, U5: TC7WB66CFK, Package_SO:VSSOP-8_2.3x2mm_P0.5mm, symbol CosmosRpiDevBoard:TC7WB66CFK
- added C10, C14, C21, C22, C23, C26, C27, C28, C30, C31, C34, C35, C36, C37, C38, C39, C41, C42, C44, C46: 100n, Capacitor_SMD:C_0402_1005Metric, symbol Device:C
- added C11, C15: 10n, Capacitor_SMD:C_0402_1005Metric, symbol Device:C
- added C12, C32, C33, C8: 10u, Capacitor_SMD:C_0402_1005Metric, symbol Device:C
- added C13, C19, C20, C24, C25, C29, C40, C43, C45, C49, C9: 1u, Capacitor_SMD:C_0402_1005Metric, symbol Device:C
- added C16: 100n, Capacitor_SMD:C_1206_3216Metric, symbol Device:C
- added C17, C18: 30p, Capacitor_SMD:C_0402_1005Metric, symbol Device:C
- added C4, C5: 6p, Capacitor_SMD:C_0402_1005Metric, symbol Device:C
- added C47, C48, C6, C7: 15p, Capacitor_SMD:C_0402_1005Metric, symbol Device:C
- added C50, C51: 3.3p, Capacitor_SMD:C_0402_1005Metric, symbol Device:C
- added J2: ARJM11D7-009-AB-EW2, ARJM11D7-009-AB-EW2:ABRACON_ARJM11D7-009-AB-EW2, symbol ARJM11D7-009-AB-EW2:ARJM11D7-009-AB-EW2
- added J3: UJ20-C-H-G-SMT-5-P16-TR, Connector_USB:USB_C_Receptacle_GCT_USB4110, symbol Connector:USB_C_Receptacle_USB2.0_14P
- added J4: MSD-4-A, PCB:MSD-4-A, symbol Connector:Micro_SD_Card_Det1
- added L1: 2.2u, PCB:L_0806_2016Metric, symbol PCM_Elektuur:L
- added L2: 2.2n, Inductor_SMD:L_0402_1005Metric, symbol PCM_Elektuur:L
- added R10, R11, R7, R8, R9: 2.2k, Resistor_SMD:R_0402_1005Metric, symbol Device:R
- added R12, R13: 220, Resistor_SMD:R_0402_1005Metric, symbol Device:R
- added R14: 12k, Resistor_SMD:R_0402_1005Metric, symbol Device:R
- added R15, R16, R17, R18, R19, R22, R23, R24, R25, R26, R27, R28, R29, R3, R30, R31, R32, R33, R34, R35, R6: 10k, Resistor_SMD:R_0402_1005Metric, symbol Device:R
- added R20, R21: 5.1k, Resistor_SMD:R_0402_1005Metric, symbol Device:R
- added R4: 6.49k, Resistor_SMD:R_0402_1005Metric, symbol Device:R
- added R5: 1M, Resistor_SMD:R_1206_3216Metric, symbol Device:R
- added SW2: DS04-254-1L-01BK, symbol Switch:SW_SPST
- added U10: 4677, Package_SO:SOIC-8_3.9x4.9mm_P1.27mm, symbol CosmosRpiDevBoard:4677
- added U11: AT25SF641B, Package_SO:SOIC-8_5.3x5.3mm_P1.27mm, symbol CosmosRpiDevBoard:AT25SF641B
- added U2: ~, PCB:PCB_Antenna, symbol CosmosRpiDevBoard:PCB_Antenna
- added U3: STM32H563RGTx, Package_QFP:LQFP-64_10x10mm_P0.5mm, symbol MCU_ST_STM32H5:STM32H563RGTx
- added U5: ESP32-S3, Package_DFN_QFN:QFN-56-1EP_7x7mm_P0.4mm_EP4x4mm, symbol MCU_Espressif:ESP32-S3
- added U6: DP83825I, Package_DFN_QFN:Texas_RMQ0024A_WQFN-24-1EP_3x3mm_P0.4mm_EP1.9x1.9mm, symbol Interface_Ethernet:DP83825I
- added U7: USB2422, Package_DFN_QFN:QFN-24-1EP_4x4mm_P0.5mm_EP2.5x2.5mm, symbol CosmosRpiDevBoard:USB2422
- added U8: PE1805, Package_TO_SOT_SMD:SOT-23-6, symbol CosmosRpiDevBoard:PE1805
- added U9: RT8010-33, PCB:RT8010, symbol CosmosRpiDevBoard:RT8010-33
- added Y1: 25MHz, Crystal:Crystal_SMD_3225-4Pin_3.2x2.5mm, symbol Device:Crystal_GND24
- added Y2: 40MHz, Crystal:Crystal_SMD_3225-4Pin_3.2x2.5mm, symbol Device:Crystal_GND24
- added Y3, Y4: 32.768kHz, symbol Device:Crystal
- C1, C3: footprint (none) -> Capacitor_SMD:C_0402_1005Metric
- R1, R2: footprint (none) -> Resistor_SMD:R_0402_1005Metric
Connections:
- net +5V: now also C31.1, C33.1, J3.A4 (VBUS), J3.A9 (VBUS), J3.B4 (VBUS), J3.B9 (VBUS), U8.5 (VCC), U9.2 (EN)
- net GND: now also C10.2, C11.2, C12.2, C13.2, C14.2, C15.2, C16.1, C17.2, C18.2, C19.2, C20.2, C21.2, C22.2, C23.2, C24.2, C25.2, C26.2, C27.2, C28.2, C29.2, C30.2, C31.2, C32.2, C33.2, C34.2, C35.2, C36.2, C37.2, C38.2, C39.2, C4.2, C40.2, C41.2, C42.2, C43.2, C44.2, C45.2, C46.2, C47.2, C48.2, C49.2, C5.2, C50.2, C51.2, C6.2, C7.2, C8.2, C9.2, J2.8 (GND), J3.A1 (GND), J3.A12 (GND), J3.B1 (GND), J3.B12 (GND), R12.2, R13.2, R14.2, R16.1, R17.1, R18.1, R19.1, R20.1, R21.1, R3.2, R34.2, R35.2, R4.2, R5.2, R6.2, SW2.1 (A), U10.4 (VSS), U11.4 (GND), U2.1, U5.57 (GND), U6.21 (GND), U6.25 (GND), U6.9 (GND), U7.25 (VSS), U8.2 (GND), U9.5 (GND), U9.7 (EP), Y1.2, Y1.4, Y2.2, Y2.4
- net +3.3V: now reaches SW1.1 (A)
- net +3.3V: now also C10.1, C11.1, C12.1, C13.1, C14.1, C15.1, C23.1, C24.1, C27.1, C28.1, C29.1, C30.1, C32.1, C34.1, C35.1, C36.1, C37.1, C38.1, C39.1, C40.1, C41.1, C42.1, C43.1, C44.1, C45.1, C46.1, C8.1, C9.1, J4.4 (VDD), L1.2 (-), R10.1, R11.1, R15.2, R23.1, R24.1, R25.1, R26.1, R27.1, R28.1, R29.1, R30.1, R31.1, R32.1, R33.1, R7.1, R8.1, R9.1, U10.8 (VCC), U11.8 (VCC), U5.2 (VDD3P3), U5.20 (VDD3P3_RTC), U5.29 (VDD_SPI), U5.3 (VDD3P3), U5.46 (VDD3P3_CPU), U5.55 (VDDA), U5.56 (VDDA), U6.19 (VDDIO), U6.6 (VDDA3V3), U7.1 (VDD33), U7.16 (VBUS_DET), U7.18 (VDD33), U7.9 (VDD33), U9.6 (FB)
- net USART_SWITCH: now reaches SW1.2 (B)
- net USART_SWITCH: now also R3.1
- new net: J2.10, R13.1
- new net: C47.1, Y4.1
- new net: C20.1, C21.1, J2.4 (CT1)
- new net: C6.1, U5.21 (XTAL_32K_P), Y3.1
- new net: C7.1, U5.22 (XTAL_32K_N), Y3.2
- new net: J4.9 (DET), R22.2
- new net: J3.B5 (CC2), R21.2
- new net: C25.1, U7.10 (CRFILT)
- new net: C49.1, R32.2, U5.4 (CHIP_PU)
- new net: C19.1, C22.1, J2.5 (CT2)
- new net: R17.2, U7.11 (PRTPWR2)
- new net: C50.1, L2.2 (-), U2.2
- new net: U3.18 (VSS), U3.31 (VSS), U3.47 (VSS), U3.63 (VSS)
- new net: R4.1, U6.14 (RBIAS)
- new net: J2.12, R12.1
- new net: J3.A5 (CC1), R20.2
- new net: R16.2, U7.17 (NON_REM0)
- new net: L1.1 (+), U9.4 (SW)
- new net: R35.1, U5.51 (GPIO45)
- new net: R34.1, U5.52 (GPIO46)
- new net: R14.1, U7.24 (RBIAS)
- new net: R6.1, U6.22 (RX_ER/S(A-MDIX))
- new net: R18.2, U7.7 (PRTPWR1)
- new net: R15.1, U7.13 (NON_REM1)
- new net: R19.2, U7.14 (CFG_SEL)
- new net: C26.1, U7.23 (PLLFILT)
- new net: C48.1, Y4.2
- new net ESP32_ANT: C51.1, L2.1 (+), U5.1 (LNA_IN)
- new net ESP32_BOOT: R33.2, SW2.2 (B), U5.5 (GPIO0)
- new net ESP32_D+: U5.26 (GPIO20/USB_D+), U7.5 (USB2_D+)
- new net ESP32_D-: U5.25 (GPIO19/USB_D-), U7.4 (USB2_D-)
- new net ESP32_RX: U5.24 (GPIO18)
- new net ESP32_TX: U5.23 (GPIO17)
- new net ESP32_XI: C4.1, U5.54 (XTAL_P), Y2.1
- new net ESP32_XO: C5.1, U5.53 (XTAL_N), Y2.3
- new net ETH_CRS_DV: R7.2, U6.20 (CRS_DV/S(PhyAdd[1]))
- new net ETH_LED_G: J2.9, U6.4 (LED0/S(ANEG_Dis))
- new net ETH_LED_Y: J2.11
- new net ETH_MDC: U6.16 (MDC)
- new net ETH_MDIO: R11.2, U6.15 (MDIO)
- new net ETH_RD+: J2.3 (RD+), U6.8 (RD+)
- new net ETH_RD-: J2.6 (RD-), U6.7 (RD-)
- new net ETH_REF_CLK: U6.2 (50MHzOut/LED2/S(RX_DV_EN))
- new net ETH_RXD_0: R9.2, U6.18 (RX_D0/S(PhyAdd[0]))
- new net ETH_RXD_1: R8.2, U6.17 (RX_D1/S(Master/Slave))
- new net ETH_TD+: J2.1 (TD+), U6.11 (TD+)
- new net ETH_TD-: J2.2 (TD-), U6.10 (TD-)
- new net ETH_TXD_0: U6.23 (TX_D0)
- new net ETH_TXD_1: U6.24 (TX_D1)
- new net ETH_TX_EN: U6.1 (TX_EN)
- new net ETH_XI: C18.1, U6.13 (XI/50MHzIn), Y1.1
- new net ETH_XO: C17.1, U6.12 (XO), Y1.3
- new net GND_CHS: C16.2, J2.SH1 (SHIELD), J2.SH2 (SHIELD__1), J3.S1 (SHIELD), J4.10 (SHIELD), R5.1
- new net INT_N: R10.2, U6.3 (INTR/~{PWRDN})
- new net RST_N: U6.5 (~{RST}), U7.15 (RESET_N)
- new net SD_CD: R22.1
- new net SD_CLK: J4.5 (CLK)
- new net SD_CMD: J4.3 (CMD), R27.2
- new net SD_DAT0: J4.7 (DAT0), R23.2
- new net SD_DAT1: J4.8 (DAT1), R24.2
- new net SD_DAT2: J4.1 (DAT2), R25.2
- new net SD_DAT3: J4.2 (DAT3/CD), R26.2
- new net SPI0_CLK: U10.6 (SCLK), U11.6 (SCK), U5.33 (SPICLK)
- new net SPI0_CS0: R31.2, U11.1 (CS#), U5.32 (SPICS0)
- new net SPI0_CS1: R30.2, U10.1 (CE#), U5.28 (SPICS1)
- new net SPI0_HD: U10.7 (IO3), U11.7 (IO3), U5.30 (SPIHD)
- new net SPI0_MISO: U10.5 (IO0), U11.5 (IO0), U5.35 (SPID)
- new net SPI0_MOSI: U10.2 (IO1), U11.2 (IO1), U5.34 (SPIQ)
- new net SPI0_WP: U10.3 (IO2), U11.3 (IO2), U5.31 (SPIWP)
- new net SPI1_CLK: U5.17 (GPIO12)
- new net SPI1_CS: R29.2, U5.15 (GPIO10)
- new net SPI1_MISO: U5.18 (GPIO13)
- new net SPI1_MOSI: U5.16 (GPIO11)
- new net SPI2_CLK: U5.13 (GPIO8)
- new net SPI2_CS: R28.2, U5.11 (GPIO6)
- new net SPI2_MISO: U5.14 (GPIO9)
- new net SPI2_MOSI: U5.12 (GPIO7)
- new net STM32_D+: U7.3 (USB1_D+)
- new net STM32_D-: U7.2 (USB1_D-)
- new net USB_CLK: U7.22 (XTALIN)
- new net USB_D+: J3.A6 (D+), J3.B6 (D+), U7.20 (USB_UP_D+), U8.1 (IO1), U8.6 (IO4)
- new net USB_D-: J3.A7 (D-), J3.B7 (D-), U7.19 (USB_UP_D-), U8.3 (IO2), U8.4 (IO3)
- no-connect marks 28 -> 52
Other:
- moved on the sheet: J1, SW1

Commit message: Update
Parts:
- removed SW1: DS04-254-1L-01BK, symbol Switch:SW_SPST
- added C52, C57, C58, C59, C60, C61, C62: 100n, Capacitor_SMD:C_0402_1005Metric, symbol Device:C
- added C53, C56: 1u, Capacitor_SMD:C_0402_1005Metric, symbol Device:C
- added C54, C55: 2.2u, Capacitor_SMD:C_0402_1005Metric, symbol Device:C
- added C63, C64: 6p, Capacitor_SMD:C_0402_1005Metric, symbol Device:C
- added D1, D2, D3, D4, D5: LED, LED_SMD:LED_0603_1608Metric, symbol Device:LED
- added H1, H2, H3, H4: Hole, PCB:RPi_Hole, symbol Mechanical:MountingHole_Pad
- added J5: 5V Fan, Connector_PinHeader_2.54mm:PinHeader_1x03_P2.54mm_Vertical, symbol Connector_Generic:Conn_01x03
- added J6: 3.3V Fan, Connector_PinHeader_2.54mm:PinHeader_1x03_P2.54mm_Vertical, symbol Connector_Generic:Conn_01x03
- added J7: Ext Pins, Connector_PinHeader_2.54mm:PinHeader_1x02_P2.54mm_Vertical, symbol Connector_Generic:Conn_01x02
- added J8: SW Debug, Connector_PinHeader_2.54mm:PinHeader_1x03_P2.54mm_Vertical, symbol Connector_Generic:Conn_01x03
- added R36: 10k, Resistor_SMD:R_0402_1005Metric, symbol Device:R
- added R37, R38, R39, R40, R41, R42, R43, R44, R45, R51: 33, Resistor_SMD:R_0402_1005Metric, symbol Device:R
- added R46, R47, R48: 100, Resistor_SMD:R_0402_1005Metric, symbol Device:R
- added R49, R50: 430, Resistor_SMD:R_0402_1005Metric, symbol Device:R
- added SW1: DS04-254-1L-03BK, Button_Switch_THT:SW_DIP_SPSTx03_Slide_6.7x9.18mm_W7.62mm_P2.54mm_LowProfile, symbol Switch:SW_DIP_x03
- added Y5: 48MHz, Crystal:Crystal_SMD_3225-4Pin_3.2x2.5mm, symbol Device:Crystal_GND24
- C2: footprint (none) -> Capacitor_SMD:CP_Elec_6.3x5.9
- J1: footprint (none) -> Connector_PinSocket_2.54mm:PinSocket_2x20_P2.54mm_Vertical
- J2: footprint ARJM11D7-009-AB-EW2:ABRACON_ARJM11D7-009-AB-EW2 -> PCB:ARJM11D7-009-AB-EW2
- SW2: value DS04-254-1L-01BK -> TS02-66-43-BK-160-LCR-D; footprint (none) -> Button_Switch_THT:SW_PUSH_6mm_H4.3mm
- Y3, Y4: footprint (none) -> Crystal:Crystal_Round_D2.0mm_Vertical
Connections:
- net USART_SWITCH is gone; now on net GND: R3.1
- net +3.3V: now also U3.1 (VBAT), U3.13 (VDDA), U3.19 (VDD), U3.32 (VDD), U3.48 (VDD), U3.64 (VDD), C56.1, C57.1, C58.1, C59.1, C60.1, C61.1, C62.1, D1.2 (A), J6.1 (Pin_1), R36.1, SW1.1, SW1.3
- net +5V: now also D2.2 (A), J5.1 (Pin_1)
- net +5V_RPi: now also D5.2 (A)
- net ESP32_BOOT: now also SW1.5; no longer SW2.2 (B)
- net ESP32_RX: now also U3.37 (PC6)
- net ESP32_TX: now also U3.38 (PC7)
- net ETH_CRS_DV: now also U3.23 (PA7)
- net ETH_LED_Y: now also U3.28 (PB2)
- net ETH_MDC: now also U3.9 (PC1)
- net ETH_MDIO: now also U3.16 (PA2)
- net ETH_REF_CLK: now also U3.15 (PA1)
- net ETH_RXD_0: now also U3.24 (PC4), R38.1; no longer U6.18 (RX_D0/S(PhyAdd[0]))
- net ETH_RXD_1: now also U3.25 (PC5), R37.1; no longer U6.17 (RX_D1/S(Master/Slave))
- net ETH_TXD_0: now also R39.2
- net ETH_TXD_1: now also R40.2
- net ETH_TX_EN: now also U3.21 (PA5)
- net GND: now also J4.10 (SHIELD), U3.12 (VSSA), U3.18 (VSS), U3.31 (VSS), U3.47 (VSS), U3.63 (VSS), C52.2, C53.2, C54.2, C55.2, C56.2, C57.2, C58.2, C59.2, C60.2, C61.2, C62.2, C63.2, C64.2, H1.1, H2.1, H3.1, H4.1, J5.3 (Pin_3), J6.3 (Pin_3), J8.3 (Pin_3), R46.2, R47.2, R48.2, R49.2, R50.2, SW1.2, Y5.2, Y5.4; no longer R3.2
- net GND_CHS: no longer J4.10 (SHIELD)
- net INT_N: now also U3.29 (PB10)
- net RPi_CTRL: now also SW1.4
- net RPi_RX: now also U3.42 (PA9)
- net RPi_TX: now also U3.43 (PA10)
- net RST_N: now also SW2.2 (B), U3.7 (NRST), C52.1, C53.1, R36.2, R41.1; no longer U6.5 (~{RST})
- net SD_CD: now also U3.50 (PA15(JTDI))
- net SD_CLK: now also U3.53 (PC12)
- net SD_CMD: now also U3.54 (PD2)
- net SD_DAT0: now also U3.39 (PC8)
- net SD_DAT1: now also U3.40 (PC9)
- net SD_DAT2: now also U3.51 (PC10)
- net SD_DAT3: now also U3.52 (PC11)
- net SPI1_CLK: now also U3.55 (PB3(JTDO)
- net SPI1_CS: now also U3.20 (PA4)
- net SPI1_MISO: now also R44.2
- net SPI1_MOSI: now also U3.57 (PB5), R43.1; no longer U5.16 (GPIO11)
- net SPI2_CLK: now also U3.34 (PB13)
- net SPI2_CS: now also U3.17 (PA3)
- net SPI2_MISO: now also R45.1
- net SPI2_MOSI: now also U3.11 (PC3), R42.1; no longer U5.12 (GPIO7)
- net STM32_D+: now also U3.45 (PA12)
- net STM32_D-: now also U3.44 (PA11)
- net USB_CLK: now also R51.2
- net ETH_LED_G_K: now reaches J2.10, R13.1
- net STM32_LXI: now reaches C47.1, Y4.1
- net STM32_LXI: now also U3.3 (PC14)
- net ETH_CT1: now reaches C20.1, C21.1, J2.4 (CT1)
- net ESP32_LXI: now reaches C6.1, U5.21 (XTAL_32K_P), Y3.1
- net ESP32_LXO: now reaches C7.1, U5.22 (XTAL_32K_N), Y3.2
- net SD_DET: now reaches J4.9 (DET), R22.2
- net USB_CC2: now reaches J3.B5 (CC2), R21.2
- net USB_CR_FILT: now reaches C25.1, U7.10 (CRFILT)
- net ESP32_CHIP_PU: now reaches C49.1, R32.2, U5.4 (CHIP_PU)
- net ETH_CT2: now reaches C19.1, C22.1, J2.5 (CT2)
- net USB_PWR2: now reaches R17.2, U7.11 (PRTPWR2)
- net ESP32_ANT_IN: now reaches C50.1, L2.2 (-), U2.2
- net STM32_SPI2_MISO: now reaches U3.10 (PC2)
- net STM32_SPI2_MISO: now also R45.2
- net STM32_WKUP: now reaches U3.14 (PA0)
- net STM32_WKUP: now also U5.7 (GPIO2)
- net STM32_SPI1_MISO: now reaches U3.22 (PA6)
- net STM32_SPI1_MISO: now also R44.1
- net STM32_VCAP1: now reaches U3.30 (VCAP)
- net STM32_VCAP1: now also C55.1
- net STM32_ETH_TX0: now reaches U3.33 (PB12)
- net STM32_ETH_TX0: now also R39.1
- net STM32_ETH_TX1: now reaches U3.36 (PB15)
- net STM32_ETH_TX1: now also R40.1
- net STM32_LXO: now reaches U3.4 (PC15)
- net STM32_LXO: now also C48.1, Y4.2
- net STM32_USB_CLK: now reaches U3.41 (PA8)
- net STM32_USB_CLK: now also R51.1
- net STM32_SWDIO: now reaches U3.46 (PA13(JTMS)
- net STM32_SWDIO: now also J8.1 (Pin_1)
- net STM32_SWCLK: now reaches U3.49 (PA14(JTCK)
- net STM32_SWCLK: now also J8.2 (Pin_2)
- net STM32_HXI: now reaches U3.5 (PH0)
- net STM32_HXI: now also C63.1, Y5.1
- net EXT_RST: now reaches U3.59 (PB7)
- net EXT_RST: now also J7.1 (Pin_1)
- net STM32_HXO: now reaches U3.6 (PH1)
- net STM32_HXO: now also C64.1, Y5.3
- net STM32_BOOT: now reaches U3.60 (BOOT0)
- net STM32_BOOT: now also R3.2, SW1.6
- net EXT_BOOT: now reaches U3.61 (PB8)
- net EXT_BOOT: now also J7.2 (Pin_2)
- net STM32_VCAP2: now reaches U3.62 (VCAP)
- net STM32_VCAP2: now also C54.1
- net ETH_BIAS: now reaches R4.1, U6.14 (RBIAS)
- net ETH_LED_Y_K: now reaches J2.12, R12.1
- net USB_CC1: now reaches J3.A5 (CC1), R20.2
- net USB_NON_REM0: now reaches R16.2, U7.17 (NON_REM0)
- net ESP32_PWM2: now reaches U5.10 (GPIO5)
- net ESP32_PWM2: now also J6.2 (Pin_2)
- net ESP32_GPIO45: now reaches R35.1, U5.51 (GPIO45)
- net ESP32_GPIO46: now reaches R34.1, U5.52 (GPIO46)
- net ESP32_LED: now reaches U5.6 (GPIO1)
- net ESP32_LED: now also D4.2 (A)
- net ESP32_PWM1: now reaches U5.9 (GPIO4)
- net ESP32_PWM1: now also J5.2 (Pin_2)
- net USB_RBIAS: now reaches R14.1, U7.24 (RBIAS)
- net ETH_RX_ER: now reaches R6.1, U6.22 (RX_ER/S(A-MDIX))
- net USB_PWR1: now reaches R18.2, U7.7 (PRTPWR1)
- net USB_NON_REM1: now reaches R15.1, U7.13 (NON_REM1)
- net USB_CFG_SEL: now reaches R19.2, U7.14 (CFG_SEL)
- net USB_PLL_FILT: now reaches C26.1, U7.23 (PLLFILT)
- net ESP32_XI renamed ESP32_HXI
- net ESP32_XO renamed ESP32_HXO
- new net: D4.1 (K), R48.1
- new net: D1.1 (K), R46.1
- new net: D2.1 (K), R49.1
- new net: D3.1 (K), R47.1
- new net: D5.1 (K), R50.1
- new net ESP32_SPI1_MOSI: R43.2, U5.16 (GPIO11)
- new net ESP32_SPI2_MOSI: R42.2, U5.12 (GPIO7)
- new net ETH_RST: R41.2, U6.5 (~{RST})
- new net ETH_RX0: R38.2, U6.18 (RX_D0/S(PhyAdd[0]))
- new net ETH_RX1: R37.2, U6.17 (RX_D1/S(Master/Slave))
- new net STM32_LED: D3.2 (A)
- no-connect marks 52 -> 54
Other:
- note added: "3.3V Fan Connector"
- note added: "5V -> 3.3V 1A"
- note added: "5V Fan Connector"
- note added: "Boot Selectors"
- note added: "Chassis Connection"
- note added: "Connectors"
- note added: "ESP32"
- note added: "ESP32 Antenna"
- note added: "ESP32 Flash"
- note added: "ESP32 IC"
- note added: "ESP32 PSRAM"
- note added: "ESP32 PullUps"
- note added: "Ethernet"
- note added: "Ethernet Connector"
- note added: "Ethernet PHY"
- note added: "Ethernet PullUps"
- note added: "External Pins Connector"
- note added: "Indication LEDs"
- note added: "MicroSD"
- note added: "MicroSD Connector"
- note added: "MicroSD PullUp"
- note added: "Raspberry Pi"
- note added: "Raspberry Pi Connector"
- note added: "Raspberry Pi Holes"
- note added: "Raspberry Pi Power Toggle"
- note added: "Reset Button"
- note added: "STM32"
- note added: "Serial Wire Debug Connector"
- note added: "Switches"
- note added: "USB"
- note added: "USB Connector"
- note added: "USB Hub"
- title: (none) -> Cosmos Dev Board
- moved on the sheet: C1, C10, C11, C12, C13, C14, C15, C16, C17, C18, C19, C2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
Changed lines of the file:
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@@
 	(generator "eeschema")
 	(generator_version "9.0")
-	(paper "A0")
+	(paper "A2")
+	(title_block
+		(title "Cosmos Dev Board")
+		(date "2025-11-09")
+		(rev "V1.0.0")
+	)

Commit message: Update
Parts:
- R5: value 1M -> 390

Commit message: Update
Parts:
- removed C16: 100n, Capacitor_SMD:C_1206_3216Metric, symbol Device:C
- removed R42, R43, R44, R45, R51: 33, Resistor_SMD:R_0402_1005Metric, symbol Device:R
- removed R5: 390, Resistor_SMD:R_1206_3216Metric, symbol Device:R
- added C65, C66: 6p, Capacitor_SMD:C_0402_1005Metric, symbol Device:C
- added Y6: 24MHz, Crystal:Crystal_SMD_3225-4Pin_3.2x2.5mm, symbol Device:Crystal_GND24
- U2: footprint PCB:PCB_Antenna -> RF_Antenna:Texas_SWRA117D_2.4GHz_Right
Connections:
- net ESP32_SPI1_MOSI is gone; now on net SPI1_MOSI: U5.16 (GPIO11)
- net ESP32_SPI2_MOSI is gone; now on net SPI2_MOSI: U5.12 (GPIO7)
- net GND_CHS is gone; now on net GND: J2.SH1 (SHIELD), J2.SH2 (SHIELD__1), J3.S1 (SHIELD)
- net STM32_SPI1_MISO is gone; now on net SPI1_MISO: U3.22 (PA6)
- net STM32_SPI2_MISO is gone; now on net SPI2_MISO: U3.10 (PC2)
- net STM32_USB_CLK is gone; now on net RPi_CTRL: U3.41 (PA8)
- net +3.3V: now also R1.2
- net +5V: now also U9.3 (VIN); no longer R1.2
- net ESP32_ANT_IN: now also U2.1; no longer U2.2
- net GND: now also J4.6 (VSS), U2.2, C65.2, C66.2, Y6.2, Y6.4; no longer U2.1
- net RPi_FAULT: now also U3.35 (PB14)
- net STM32_LED: now also U3.58 (PB6)
- net USB_CLK_OUT: now reaches U7.21 (XTALOUT)
- net USB_CLK_OUT: now also C66.1, Y6.3
- net USB_CLK renamed USB_CLK_IN
- net USB_CLK_IN: now also C65.1, Y6.1
- no-connect marks 54 -> 52
Other:
- note added: "USB Crystal"
- note removed: "Chassis Connection"
- moved on the sheet: C23, C24, C25, C26, C27, C28, J3, R10, R11, R14, R15, R16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
